Commit message: finish digital twins

File: install/chan/share/chan/config/tongquan_sldasm.ros2_control.xacro (robot description, xacro)
@@ -1,40 +1 @@
-<?xml version="1.0"?>
-<robot xmlns:xacro="http://www.ros.org/wiki/xacro">
-    <xacro:macro name="tongquan_sldasm_ros2_control" params="name initial_positions_file">
-        <xacro:property name="initial_positions" value="${load_yaml(initial_positions_file)['initial_positions']}"/>
-        <ros2_control name="${name}" type="system">
-            <hardware>
-                <!-- By default, set up controllers for simulation. This won't work on real hardware -->
-                <plugin>mock_components/GenericSystem</plugin>
-            </hardware>
-            <joint name="joint_3">
-                <command_interface name="position"/>
-                <state_interface name="position">
-                  <param name="initial_value">${initial_positions['joint_3']}</param>
-                </state_interface>
-                <state_interface name="velocity"/>
-            </joint>
-            <joint name="joint_4">
-                <command_interface name="position"/>
-                <state_interface name="position">
-                  <param name="initial_value">${initial_positions['joint_4']}</param>
-                </state_interface>
-                <state_interface name="velocity"/>
-            </joint>
-            <joint name="joint_1">
-                <command_interface name="position"/>
-                <state_interface name="position">
-                  <param name="initial_value">${initial_positions['joint_1']}</param>
-                </state_interface>
-                <state_interface name="velocity"/>
-            </joint>
-            <joint name="joint_2">
-                <command_interface name="position"/>
-                <state_interface name="position">
-                  <param name="initial_value">${initial_positions['joint_2']}</param>
-                </state_interface>
-                <state_interface name="velocity"/>
-            </joint>
-        </ros2_control>
-    </xacro:macro>
-</robot>
+/home/logan/exos_new_ws/src/chan/config/tongquan_sldasm.ros2_control.xacro

File: install/chan/share/chan/config/tongquan_sldasm.urdf.xacro (robot description, xacro)
@@ -1,9 +1 @@
-<?xml version="1.0"?>
-<robot xmlns:xacro="http://www.ros.org/wiki/xacro" name="tongquan_sldasm">
-    <xacro:arg name="initial_positions_file" default="initial_positions.yaml" />
-    <!-- Import tongquan_sldasm urdf file -->
-    <xacro:include filename="$(find tongquan_sldasm)/urdf/tongquan_sldasm.urdf" />
-    <!-- Import control_xacro -->
-    <xacro:include filename="tongquan_sldasm.ros2_control.xacro" />
-    <xacro:tongquan_sldasm_ros2_control name="FakeSystem" initial_positions_file="$(arg initial_positions_file)"/>
-</robot>
+/home/logan/exos_new_ws/src/chan/config/tongquan_sldasm.urdf.xacro

File: install/moveit/share/moveit/config/tongquan_sldasm.ros2_control.xacro (robot description, xacro)
@@ -1,40 +1 @@
-<?xml version="1.0"?>
-<robot xmlns:xacro="http://www.ros.org/wiki/xacro">
-    <xacro:macro name="tongquan_sldasm_ros2_control" params="name initial_positions_file">
-        <xacro:property name="initial_positions" value="${load_yaml(initial_positions_file)['initial_positions']}"/>
-        <ros2_control name="${name}" type="system">
-            <hardware>
-                <!-- By default, set up controllers for simulation. This won't work on real hardware -->
-                <plugin>mock_components/GenericSystem</plugin>
-            </hardware>
-            <joint name="joint_1">
-                <command_interface name="position"/>
-                <state_interface name="position">
-                  <param name="initial_value">${initial_positions['joint_1']}</param>
-                </state_interface>
-                <state_interface name="velocity"/>
-            </joint>
-            <joint name="joint_2">
-                <command_interface name="position"/>
-                <state_interface name="position">
-                  <param name="initial_value">${initial_positions['joint_2']}</param>
-                </state_interface>
-                <state_interface name="velocity"/>
-            </joint>
-            <joint name="joint_3">
-                <command_interface name="position"/>
-                <state_interface name="position">
-                  <param name="initial_value">${initial_positions['joint_3']}</param>
-                </state_interface>
-                <state_interface name="velocity"/>
-            </joint>
-            <joint name="joint_4">
-                <command_interface name="position"/>
-                <state_interface name="position">
-                  <param name="initial_value">${initial_positions['joint_4']}</param>
-                </state_interface>
-                <state_interface name="velocity"/>
-            </joint>
-        </ros2_control>
-    </xacro:macro>
-</robot>
+/home/logan/exos_new_ws/src/moveit/config/tongquan_sldasm.ros2_control.xacro

File: install/moveit/share/moveit/config/tongquan_sldasm.urdf.xacro (robot description, xacro)
@@ -1,9 +1 @@
-<?xml version="1.0"?>
-<robot xmlns:xacro="http://www.ros.org/wiki/xacro" name="tongquan_sldasm">
-    <xacro:arg name="initial_positions_file" default="initial_positions.yaml" />
-    <!-- Import tongquan_sldasm urdf file -->
-    <xacro:include filename="$(find tongquan_sldasm)/urdf/tongquan_sldasm.urdf" />
-    <!-- Import control_xacro -->
-    <xacro:include filename="tongquan_sldasm.ros2_control.xacro" />
-    <xacro:tongquan_sldasm_ros2_control name="FakeSystem" initial_positions_file="$(arg initial_positions_file)"/>
-</robot>
+/home/logan/exos_new_ws/src/moveit/config/tongquan_sldasm.urdf.xacro

File: install/moveit_2/share/moveit_2/config/tongquan_sldasm.ros2_control.xacro (robot description, xacro)
@@ -1,40 +1 @@
-<?xml version="1.0"?>
-<robot xmlns:xacro="http://www.ros.org/wiki/xacro">
-    <xacro:macro name="tongquan_sldasm_ros2_control" params="name initial_positions_file">
-        <xacro:property name="initial_positions" value="${load_yaml(initial_positions_file)['initial_positions']}"/>
-        <ros2_control name="${name}" type="system">
-            <hardware>
-                <!-- By default, set up controllers for simulation. This won't work on real hardware -->
-                <plugin>mock_components/GenericSystem</plugin>
-            </hardware>
-            <joint name="joint_1">
-                <command_interface name="position"/>
-                <state_interface name="position">
-                  <param name="initial_value">${initial_positions['joint_1']}</param>
-                </state_interface>
-                <state_interface name="velocity"/>
-            </joint>
-            <joint name="joint_2">
-                <command_interface name="position"/>
-                <state_interface name="position">
-                  <param name="initial_value">${initial_positions['joint_2']}</param>
-                </state_interface>
-                <state_interface name="velocity"/>
-            </joint>
-            <joint name="joint_3">
-                <command_interface name="position"/>
-                <state_interface name="position">
-                  <param name="initial_value">${initial_positions['joint_3']}</param>
-                </state_interface>
-                <state_interface name="velocity"/>
-            </joint>
-            <joint name="joint_4">
-                <command_interface name="position"/>
-                <state_interface name="position">
-                  <param name="initial_value">${initial_positions['joint_4']}</param>
-                </state_interface>
-                <state_interface name="velocity"/>
-            </joint>
-        </ros2_control>
-    </xacro:macro>
-</robot>
+/home/logan/exos_new_ws/src/moveit_2/config/tongquan_sldasm.ros2_control.xacro

File: install/moveit_2/share/moveit_2/config/tongquan_sldasm.urdf.xacro (robot description, xacro)
@@ -1,9 +1 @@
-<?xml version="1.0"?>
-<robot xmlns:xacro="http://www.ros.org/wiki/xacro" name="tongquan_sldasm">
-    <xacro:arg name="initial_positions_file" default="initial_positions.yaml" />
-    <!-- Import tongquan_sldasm urdf file -->
-    <xacro:include filename="$(find tongquan_sldasm)/urdf/tongquan_sldasm.urdf" />
-    <!-- Import control_xacro -->
-    <xacro:include filename="tongquan_sldasm.ros2_control.xacro" />
-    <xacro:tongquan_sldasm_ros2_control name="FakeSystem" initial_positions_file="$(arg initial_positions_file)"/>
-</robot>
+/home/logan/exos_new_ws/src/moveit_2/config/tongquan_sldasm.urdf.xacro

File: install/moveit_true/share/moveit_true/config/tongquan_sldasm.ros2_control.xacro (robot description, xacro)
@@ -1,40 +1 @@
-<?xml version="1.0"?>
-<robot xmlns:xacro="http://www.ros.org/wiki/xacro">
-    <xacro:macro name="tongquan_sldasm_ros2_control" params="name initial_positions_file">
-        <xacro:property name="initial_positions" value="${load_yaml(initial_positions_file)['initial_positions']}"/>
-        <ros2_control name="${name}" type="system">
-            <hardware>
-                <!-- By default, set up controllers for simulation. This won't work on real hardware -->
-                <plugin>mock_components/GenericSystem</plugin>
-            </hardware>
-            <joint name="joint_1">
-                <command_interface name="position"/>
-                <state_interface name="position">
-                  <param name="initial_value">${initial_positions['joint_1']}</param>
-                </state_interface>
-                <state_interface name="velocity"/>
-            </joint>
-            <joint name="joint_2">
-                <command_interface name="position"/>
-                <state_interface name="position">
-                  <param name="initial_value">${initial_positions['joint_2']}</param>
-                </state_interface>
-                <state_interface name="velocity"/>
-            </joint>
-            <joint name="joint_3">
-                <command_interface name="position"/>
-                <state_interface name="position">
-                  <param name="initial_value">${initial_positions['joint_3']}</param>
-                </state_interface>
-                <state_interface name="velocity"/>
-            </joint>
-            <joint name="joint_4">
-                <command_interface name="position"/>
-                <state_interface name="position">
-                  <param name="initial_value">${initial_positions['joint_4']}</param>
-                </state_interface>
-                <state_interface name="velocity"/>
-            </joint>
-        </ros2_control>
-    </xacro:macro>
-</robot>
+/home/logan/exos_new_ws/src/moveit_true/config/tongquan_sldasm.ros2_control.xacro

File: install/moveit_true/share/moveit_true/config/tongquan_sldasm.urdf.xacro (robot description, xacro)
@@ -1,9 +1 @@
-<?xml version="1.0"?>
-<robot xmlns:xacro="http://www.ros.org/wiki/xacro" name="tongquan_sldasm">
-    <xacro:arg name="initial_positions_file" default="initial_positions.yaml" />
-    <!-- Import tongquan_sldasm urdf file -->
-    <xacro:include filename="$(find tongquan_sldasm)/urdf/tongquan_sldasm.urdf" />
-    <!-- Import control_xacro -->
-    <xacro:include filename="tongquan_sldasm.ros2_control.xacro" />
-    <xacro:tongquan_sldasm_ros2_control name="FakeSystem" initial_positions_file="$(arg initial_positions_file)"/>
-</robot>
+/home/logan/exos_new_ws/src/moveit_true/config/tongquan_sldasm.urdf.xacro
