Commit message: Let's start digital twins

File: src/tongquan_sldasm/urdf/tongquan_sldasm.urdf (robot description, URDF)
Before this commit: robot tongquan_sldasm, 5 links, 4 joints
Joints:
- joint joint_1: limit lower=-0.93 upper=0 effort=10 velocity=0.2 -> lower=-0.93 upper=0 effort=300 velocity=0.2
- joint joint_2: limit lower=0 upper=0.93 effort=10 velocity=0.2 -> lower=0 upper=0.93 effort=300 velocity=0.2
- joint joint_3: limit lower=-0.93 upper=0 effort=10 velocity=0.2 -> lower=-0.93 upper=0 effort=300 velocity=0.2
- joint joint_4: limit lower=0 upper=0.93 effort=10 velocity=0.2 -> lower=0 upper=0.93 effort=300 velocity=0.2

Commit message: Author: Logan Ngo

File: src/tongquan_sldasm/urdf/tongquan_sldasm.urdf (robot description, URDF)
Before this commit: robot tongquan_sldasm, 5 links, 4 joints
Joints:
- joint joint_1: limit lower=-0.93 upper=0 effort=300 velocity=0.2 -> lower=-0.93 upper=0 effort=30 velocity=0.5
- joint joint_2: limit lower=0 upper=0.93 effort=300 velocity=0.2 -> lower=0 upper=0.93 effort=30 velocity=0.5
- joint joint_3: limit lower=-0.93 upper=0 effort=300 velocity=0.2 -> lower=-0.93 upper=0 effort=30 velocity=0.5
- joint joint_4: limit lower=0 upper=0.93 effort=300 velocity=0.2 -> lower=0 upper=0.93 effort=30 velocity=0.5
